Commit message: 圆柱方块+导航调参+碰撞检测：房间导航 4/4、对齐 100%
- world: number1~4 由立方体网格改为等大圆柱（r0.25/h0.5，中心不变），消除立方体角导致的建图/卡死问题
- nav2_params: SmacPlanner2D、膨胀 0.40/0.45、足迹 0.25 方框、进度检查 0.15m/30s、
  RPP 碰撞前瞻 0.3s、AMCL update_min_d/a=0、到点容差 0.15m/0.20rad
- URDF: 增加 base_link 接触传感器 /bumper_states（客观碰撞计数）
- scripts: 新增 check_nav_rooms.py；check_alignment.py 增加 ±1 格容差
- maps: 圆柱版新地图（用户遥控重建，对齐 100%，4/4 到点、0 碰撞）
- docs: DEV_LOG 记录修复过程与证据

File: TestRobot/src/urdf/plugins/gazebo_control_plugin.xacro (robot description, xacro)
@@ -129,4 +129,21 @@
             </sensor>
         </gazebo>
+        <!-- ===== 碰撞检测（验收要求「全程碰撞次数少于 2 次」的客观依据） =====
+             发布话题：/bumper_states（gazebo_msgs/ContactsState）
+             仅统计车体（base_link_collision）的接触，不含轮子/万向轮与地面的正常接触 -->
+        <gazebo reference="base_link">
+            <sensor name="bumper" type="contact">
+                <update_rate>20</update_rate>
+                <contact>
+                    <collision>base_link_collision</collision>
+                </contact>
+                <plugin name="bumper_controller" filename="libgazebo_ros_bumper.so">
+                    <ros>
+                        <namespace>/</namespace>
+                    </ros>
+                    <frame_name>base_link</frame_name>
+                </plugin>
+            </sensor>
+        </gazebo>
     </xacro:macro>
 </robot>
